File: Mixer.kicad_sch (KiCad schematic)
At the start: 7 parts, among them U2 RC4558

Commit message: finalise schems for now
Parts:
- removed C34: 220n, symbol Device:C
- removed Tone: 10k, symbol Device:R_Potentiometer
- C15: footprint (none) -> Capacitor_SMD:C_0805_2012Metric
- MIX1: renamed from MIX; footprint (none) -> Potentiometer_THT:Potentiometer_Alpha_RD902F-40-00D_Dual_Vertical
- R17, R26: footprint (none) -> Resistor_SMD:R_0805_2012Metric
- U2: footprint (none) -> Package_SO:SOIC-8W_5.3x5.3mm_P1.27mm
