File: Power.kicad_sch (KiCad schematic)
At the start: 21 parts, among them U2 RC4558, U3 MC78L05_SOT89, U4 RC4558

Commit message: finalise schems for now
Parts:
- removed unit 2 of U4
- added POWER1: Conn_01x02, Connector_PinHeader_2.54mm:PinHeader_1x02_P2.54mm_Vertical, symbol Connector_Generic:Conn_01x02
- C12, C16, C17, C18, C19, C20, C21, C22, C23, C24, C25, C26, C27, C28: footprint (none) -> Capacitor_SMD:C_0805_2012Metric
- R11, R12, R18, R19: footprint (none) -> Resistor_SMD:R_0805_2012Metric
- U2, U4: footprint (none) -> Package_SO:SOIC-8W_5.3x5.3mm_P1.27mm
Connections:
- net +9V: now also POWER1.1 (Pin_1)
- net GND: now also POWER1.2 (Pin_2)
- net VREF_A: now also C16.2, C17.2, R11.1, R12.2
