File: Preamp.kicad_sch (KiCad schematic)
At the start: 18 parts, among them U4 RC4558

Commit message: finalise schems for now
Parts:
- added C35: 100p, Capacitor_SMD:C_0805_2012Metric, symbol Device:C
- added C36: 1u, Capacitor_SMD:C_0805_2012Metric, symbol Device:C
- added R27: 4k7, Resistor_SMD:R_0805_2012Metric, symbol Device:R
- added R28: 3k3, Resistor_SMD:R_0805_2012Metric, symbol Device:R
- added R29: 25k, Resistor_SMD:R_0805_2012Metric, symbol Device:R
- added Tone1: 10k, Potentiometer_THT:Potentiometer_Alpha_RD902F-40-00D_Dual_Vertical, symbol Device:R_Potentiometer
- added unit 2 of U4
- C29, C31, C32: footprint (none) -> Capacitor_SMD:C_0805_2012Metric
- C30: value 100n -> 100p; footprint (none) -> Capacitor_SMD:C_0805_2012Metric
- C33: value 10n -> 68n; footprint (none) -> Capacitor_SMD:C_0805_2012Metric
- D2, D3, D4, D5, D6: footprint (none) -> Diode_SMD:D_0603_1608Metric
- R20, R21, R22, R23, R24: footprint (none) -> Resistor_SMD:R_0805_2012Metric
- R25: value 4k7 -> 680r; footprint (none) -> Resistor_SMD:R_0805_2012Metric
- Saturation1: renamed from Saturation; footprint (none) -> Potentiometer_THT:Potentiometer_Alpha_RD902F-40-00D_Dual_Vertical
- U4: footprint (none) -> Package_SO:SOIC-8W_5.3x5.3mm_P1.27mm
Connections:
- net PRE_OUT: now also C35.2, R27.2, U4.7; no longer C33.2, R25.2
- net VREF_A: now also C36.2, R28.2
- new net: C35.1, R27.1, R28.1, R29.1, U4.6 (-)
- new net: C36.1, R29.2
- new net: R25.2, Tone1.1, Tone1.2
- new net: C33.2, Tone1.3, U4.5 (+)
Other:
- moved on the sheet: C33
