File: lofi-chorus.kicad_sch (KiCad schematic)
At the start: 0 parts

Commit message: finalise schems for now
Parts:
- added CHORUS_IN1, CHORUS_OUT1, PRE_IN1, PRE_OUT1: Conn_01x02, Connector_PinHeader_2.54mm:PinHeader_1x02_P2.54mm_Vertical, symbol Connector_Generic:Conn_01x02
Connections:
- net Mixer/DRY_IN: now also CHORUS_IN1.1 (Pin_1)
- net Mixer/MIXED_OUT: now also CHORUS_OUT1.1 (Pin_1)
- net Preamp/PRE_IN: now also PRE_IN1.1 (Pin_1)
- new net GND: CHORUS_IN1.2 (Pin_2), CHORUS_OUT1.2 (Pin_2), PRE_IN1.2 (Pin_2), PRE_OUT1.2 (Pin_2)
- new net Preamp/PRE_OUT: PRE_OUT1.1 (Pin_1)
